Commit message: changed name of frame to camera_link as realsense node publishes

File: nfr_charged_up/config/squishy.urdf (robot description, URDF)
Before this commit: robot squishy, 2 links, 1 joints
Links:
- removed link realsense
- added link camera_link
Joints:
- joint realsense_joint: child realsense -> camera_link
