Commit message: Worked on it. LOTS OF PROGRESS

File: nfr_crescendo/config/swervy.urdf (robot description, URDF)
Before this commit: robot swervy, 2 links, 1 joints
Links:
- removed link camera_link
- added link camera
Joints:
- removed joint realsense_joint
- added joint usb_camera_joint: type fixed, parent base_link, child camera, origin xyz=0.405 0 0.18 rpy=0 0 90

Commit message: TMP

File: nfr_crescendo/config/swervy.urdf (robot description, URDF)
Before this commit: robot swervy, 2 links, 1 joints
Joints:
- joint usb_camera_joint: origin xyz=0.405 0 0.18 rpy=0 0 90 -> xyz=0.405 0 0.18 rpy=0 0 0

Commit message: Still need to figure out time sync

File: nfr_crescendo/config/swervy.urdf (robot description, URDF)
Before this commit: robot swervy, 2 links, 1 joints
Links:
- removed link camera
- added link camera_link
Joints:
- joint usb_camera_joint: child camera -> camera_link

Commit message: Get working pose estimation & depth estimation (#7)
* TMP

* Finally got pose estimation mostly working

* Redid nfr_apriltag so that it was independent of apriltag_ros

* Multitag PnP worksgit add nfr_apriltag/!

* Working on nfr_bridge node

* TMPgit add -A!

* Fix AprilTagNode

* TMP

* Some change???

* Lots of changes

* TMP

* Still need to figure out time sync

* did some stuff

* Depth finder kinda works

* Lots of fixes

* Depth accuracy + pose esitmation

* Minor changes

* Reorganize everything into more nodes

File: nfr_crescendo/config/swervy.urdf (robot description, URDF)
Before this commit: robot swervy, 2 links, 1 joints
Links:
- removed link camera
- added link camera_link
Joints:
- joint usb_camera_joint: child camera -> camera_link; origin xyz=0.405 0 0.18 rpy=0 0 90 -> xyz=0.405 0 0.18 rpy=0 0 0
