Commit message: IMPORTANT FIXES + other cmaera + crabby

File: nfr_crescendo/config/crabby.urdf (robot description, URDF)
Before this commit: robot swervy, 3 links, 2 joints
Joints:
- joint realsense_camera_joint: origin xyz=0.405 0 0.18 rpy=0 0 0 -> xyz=0.2413 0 0.6604 rpy=0 0 0
- joint usb_camera_joint: origin xyz=0.405 0.1524 0.18 rpy=0 0 0 -> xyz=0.2413 0.0712 0.6604 rpy=0 0 0

Commit message: Will rename later

File: nfr_crescendo/config/crabby.urdf (robot description, URDF)
Before this commit: robot swervy, 3 links, 2 joints
Links:
- removed link camera_link
Joints:
- removed joint realsense_camera_joint
- joint usb_camera_joint: origin xyz=0.2413 0.0712 0.6604 rpy=0 0 0 -> xyz=0.2413 0 0.6604 rpy=0 0 0

File: nfr_crescendo/config/swervy.urdf (robot description, URDF)
Before this commit: robot swervy, 3 links, 2 joints
Links:
- removed link camera_link
Joints:
- removed joint realsense_camera_joint
- joint usb_camera_joint: origin xyz=0.405 0.1524 0.18 rpy=0 0 0 -> xyz=0.405 0 0.1292 rpy=0 0 0
